File: am3352_som/am3352_som.sch (KiCad schematic (older format))
At the start: 0 parts

Commit message: datasheet
Changed lines of the file:
@@
 $Descr A4 11693 8268
 encoding utf-8
-Sheet 1 2
+Sheet 1 3
 Title ""
 Date ""
@@
 F1 "som_sodimm.sch" 50
 $EndSheet
+$Sheet
+S 7650 3150 700  1600
+U 60ABBC64
+F0 "Sheet60ABBC63" 50
+F1 "rtl8211e.sch" 50
+$EndSheet
 $EndSCHEMATC

Commit message: adjust
Changed lines of the file:
@@
 $EndSheet
 $Sheet
-S 7650 3150 700  1600
+S 7200 2700 700  1600
 U 60ABBC64
 F0 "Sheet60ABBC63" 50

Commit message: pre
Changed lines of the file:
@@
 $Descr A4 11693 8268
 encoding utf-8
-Sheet 1 3
+Sheet 1 4
 Title ""
 Date ""
@@
 F1 "rtl8211e.sch" 50
 $EndSheet
+$Sheet
+S 3400 2600 1400 1900
+U 60B42247
+F0 "Sheet60B42246" 50
+F1 "peripheral.sch" 50
+$EndSheet
 $EndSCHEMATC
